File: ControllerCircuit/ControllerCircuit.kicad_pcb (KiCad board)
At the start: 2 copper layers, 122.5 x 87.5 mm, 87 parts, among them J1 ScrewTerminal, J10 Conn_01x02_Female, J11 Conn_01x03_Female, J12 ScrewTerminal, J13 Conn_01x02_Female, J14 ScrewTerminal, J15 Molex 0472192001, J2 ScrewTerminal3Pin, J3 ScrewTerminal3Pin, J4 ScrewTerminal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

Commit message: test commit
Parts:
- added JP6: A0 Volt Select, Jumper:SolderJumper-3_P1.3mm_Bridged12_RoundedPad1.0x1.5mm, F.Cu at (148.2, 112.0)
- added JP7: I/O Volt Select, Jumper:SolderJumper-3_P1.3mm_Bridged12_RoundedPad1.0x1.5mm, F.Cu at (153.7, 112.2)
- added Q4: AO3400A, Package_TO_SOT_SMD:SOT-23, F.Cu at (175.8, 120.2)
- added R7: 2K2, Resistor_SMD:R_0805_2012Metric, F.Cu at (176.4, 123.8)
- R2: value 2K2 -> 1M
- U3: value TCA6408APWR -> PCA9538PW,118
- moved C6 9.48 mm to (152.5, 123.6), turned to 180 degrees
- moved R2 6.64 mm to (176.8, 116.8)
- moved R24 0.79 mm to (123.9, 127.4)
- moved R5 0.12 mm to (101.2, 62.6)
- moved R16 0.05 mm to (101.2, 60.3)
Connections:
- C6 pad 1: +3V3 -> /U3_PWR
- J15 pad 1: (no net) -> Net-(J15-Pad1)
- J15 pad 8: (no net) -> Net-(J15-Pad8)
- R2 pad 1: GND -> /IO2
- R2 pad 2: /IO2 -> +3V3
- RX1 pad 1: /IO2 -> GND
- RX1 pad 2: +3V3 -> Net-(Q4-Pad1)
- U3 pad 1: +3V3 -> Net-(JP6-Pad2)
- U3 pad 16: FUSED5V -> /U3_PWR
- U4 pad 1: (no net) -> /ESP3V3
- U4 pad 16: (no net) -> Net-(U4-Pad16)
- U4 pad 17: (no net) -> Net-(U4-Pad17)
- U4 pad 18: (no net) -> Net-(U4-Pad18)
- U4 pad 23: (no net) -> Net-(U4-Pad23)
- U4 pad 24: (no net) -> Net-(U4-Pad24)
- U4 pad 36: (no net) -> Net-(U4-Pad36)
- U4 pad 37: (no net) -> Net-(U4-Pad37)
- U4 pad 38: (no net) -> Net-(U4-Pad38)
Routing:
- net /U3_PWR: track 0.00 -> 18.5 mm, vias 0 -> 2
- net /IO2: track 80.5 -> 67.8 mm
- net GND: track 42.5 -> 52.9 mm, vias 236 -> 245
- net Net-(Q4-Pad1): track 0.00 -> 9.90 mm
- net Net-(JP6-Pad2): track 0.00 -> 6.08 mm
- net +3V3: track 394.2 -> 390.1 mm, vias 10 -> 14
- net /IO27: track 213.4 -> 210.0 mm
- net FUSED5V: track 299.4 -> 296.4 mm
- net /IO26: track 194.3 -> 191.6 mm
- net /RESET: track 144.2 -> 146.5 mm
- net /IO39_INPUT: track 95.8 -> 94.1 mm
- net /CANBUS_RX: track 63.8 -> 65.4 mm
- net /IO22: track 65.4 -> 63.9 mm
- net /VSPI_CLK: track 161.0 -> 162.3 mm
- net /IO35_INPUT: track 116.8 -> 118.0 mm
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